Commit message: feat(emotion-sim): emotion engine, 3D sim, and dashboard integration
- Add 4-axis emotion engine to NeoDM (energy, valence, arousal, anxiety)
- Implement EmotionSim.svelte: Three.js GLB viewer with per-zone touch detection
  (Ear, Head, Face, Nose, Arm, Belly, Back) and real-time emotion parameter updates
- Add Map / Emotion Sim tab switcher to dashboard header
- Fix foxglove-bridge: GLB/STL HTTP serving, fetchAsset WebSocket protocol, robot.urdf
- Fix behavior.go gRPC DNS resolution (dns:/// prefix for Docker)
- Fix dashboard redis.go: GetLabel → GetEyeState
- Add three@0.128.0 dependency to dashboard frontend
- Gitignore model mesh assets and compiled binaries
- Update README: Emotion Sim usage, robot model setup guide, updated roadmap

File: middleware/services/foxglove-bridge/robot.urdf (robot description, URDF)
Before this commit: robot robotos, 10 links, 9 joints
Links:
- removed link body_bottom_link
- removed link caster_link
- removed link head_link
- removed link horn_base_link
- removed link horn_tip_link
- removed link left_flipper_link
- removed link left_wheel_link
- removed link right_flipper_link
- removed link right_wheel_link
- link base_link: mass None -> 2.0; geometry collision box size=0.21 0.15 0.35; visual mesh filename=http://localhost:8765/meshes/bunny.stl
Joints:
- removed joint body_bottom_joint
- removed joint caster_joint
- removed joint head_joint
- removed joint horn_base_joint
- removed joint horn_tip_joint
- removed joint left_flipper_joint
- removed joint left_wheel_joint
- removed joint right_flipper_joint
- removed joint right_wheel_joint
